File: FPGA-Lockin.kicad_pcb (KiCad board)
At the start: 4 copper layers, 48.8 x 55.2 mm, 124 parts, among them J1 SPI Header, J2 G125-MH104M4-04AD000P, J3 Laser, J4 PZT, J5 Micro_SD_Card, J6 Conn_02x07_Odd_Even, J7 Conn_01x02_Pin, U1 ICE40UP5K-SG48ITR, U10 OPA310xDBV, U11 MCP1501-30xSN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

Commit message: Fix everything based on component availabilty
Parts:
- removed C6: 1uF, Capacitor_SMD:C_0805_2012Metric_Pad1.18x1.45mm_HandSolder
- added C21: 120uF, Capacitor_Tantalum_SMD:CP_EIA-7132-20_AVX-U_HandSolder, F.Cu at (119.6, 49.7)
- added C45: 0.1uF, Capacitor_SMD:C_0805_2012Metric_Pad1.18x1.45mm_HandSolder, B.Cu at (125.4, 48.4)
- added L3: 1uH, Inductor_SMD:L_1206_3216Metric_Pad1.22x1.90mm_HandSolder, B.Cu at (147.0, 72.8)
- added R25: 10kR, Resistor_SMD:R_0805_2012Metric_Pad1.20x1.40mm_HandSolder, F.Cu at (115.4, 49.4)
- added R26: 100kR, Resistor_SMD:R_0805_2012Metric_Pad1.20x1.40mm_HandSolder, B.Cu at (152.0, 72.6)
- added R27: 100kR, Resistor_SMD:R_0805_2012Metric_Pad1.20x1.40mm_HandSolder, B.Cu at (151.2, 75.8)
- C4: value 1uF -> 4.7uF
- C43: value 0.1uF -> 1uF
- C5: value 10nF -> 22uF
- U14: value MIC94090YC6 -> AP22802AW5-7; footprint Package_TO_SOT_SMD:SOT-363_SC-70-6 -> switch:SOT25_DIO
- U3: value SPX3819M5-L-1-2 -> TLV62568ADRL; footprint Package_TO_SOT_SMD:SOT-23-5 -> Package_TO_SOT_SMD:SOT-563
- moved C5 10.8 mm to (144.8, 69.6), turned to 90 degrees
- moved C4 8.38 mm to (144.4, 78.0), turned to -90 degrees
- moved J7 3.58 mm to (123.8, 53.5)
- moved C3 3.23 mm to (148.6, 78.2)
- moved U3 1.30 mm to (145.5, 75.0), turned to 180 degrees
- moved U14 0.32 mm to (124.4, 46.6)
Connections:
- C4 pad 1: +2V5 -> +5V
- C5 pad 1: Net-(U3-BP) -> +1V2
- U14 pad 3: unconnected-(U14-NC-Pad3) -> Net-(U14-FLG)
- U14 pad 4: +5V -> /LSR_ON
- U14 pad 5: GND -> +5V
- U3 pad 1: +2V5 -> Net-(U3-FB)
- U3 pad 3: +2V5 -> +5V
- U3 pad 4: Net-(U3-BP) -> Net-(U3-SW)
- U3 pad 5: +1V2 -> +5V
Routing:
- net +2V5: track 69.3 -> 58.2 mm
- net +5V: track 64.3 -> 75.3 mm, vias 9 -> 12
- net Net-(U3-FB): track 0.00 -> 9.04 mm
- net Net-(JP2-A): track 3.34 -> 11.6 mm
- net Net-(U14-FLG): track 0.00 -> 7.88 mm
- net +1V2: track 45.4 -> 52.5 mm
- net GND: track 149.5 -> 154.3 mm
- net Net-(U3-SW): track 0.00 -> 4.33 mm
- net Net-(U3-BP): track 2.71 -> 0.00 mm
- net GNDA: track 82.9 -> 84.5 mm
