File: can.kicad_sch (KiCad schematic)
At the start: 9 parts, among them J5 Micro_SD_Card, U15 MCP2562, Y1 Crystal_GND24

Commit message: Fix review suggestions from non-fpga board
Parts:
- C30, C31: value 27pF -> 10pF
- Y1: value Crystal_GND24 -> ABM8G
Connections:
- net SS1_mem renamed ~{SS1_mem}
Changed lines of the file:
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@@
-	(wire
-		(pts
-			(xy 195.58 101.6) (xy 194.31 101.6)
-		)
-		(stroke
-			(width 0)
-			(type default)
-		)
-	)
 	(wire
 		(pts
@@
 		)
 	)
-	(hierarchical_label "SS1_mem"
+	(hierarchical_label "~{SS1_mem}"
 		(shape input)
 		(at 166.37 77.47 180)
@@
 	(symbol
 		(lib_id "power:GND")
-		(at 194.31 101.6 0)
+		(at 195.58 101.6 0)
 		(unit 1)
 		(exclude_from_sim no)
@@
 		(fields_autoplaced yes)
 		(property "Reference" "#PWR077"
-			(at 194.31 107.95 0)
+			(at 195.58 107.95 0)
 			(effects
 				(font
@@
 		)
 		(property "Value" "GND"
-			(at 194.31 106.68 0)
+			(at 195.58 106.68 0)
 			(effects
 				(font
@@
 		)
 		(property "Footprint" ""
-			(at 194.31 101.6 0)
+			(at 195.58 101.6 0)
 			(effects
 				(font
@@
 		)
 		(property "Datasheet" ""
-			(at 194.31 101.6 0)
+			(at 195.58 101.6 0)
 			(effects
 				(font
@@
 		)
 		(property "Description" "Power symbol creates a global label with name \"GND\" , ground"
-			(at 194.31 101.6 0)
+			(at 195.58 101.6 0)
 			(effects
 				(font
@@
 			)
 		)
-		(property "Value" "27pF"
+		(property "Value" "10pF"
 			(at 38.1 50.8 90)
 			(effects
@@
 			)
 		)
-		(property "Value" "27pF"
+		(property "Value" "10pF"
 			(at 38.1 63.5 90)
 			(effects
@@
 			)
 		)
-		(property "Value" "Crystal_GND24"
+		(property "Value" "ABM8G"
 			(at 55.88 63.4999 90)
 			(effects
@@
 			)
 		)
-		(property "Datasheet" "~"
+		(property "Datasheet" "https://abracon.com/Resonators/ABM8G.pdf"
 			(at 60.96 62.23 0)
 			(effects
