File: power.kicad_sch (KiCad schematic)
At the start: 36 parts, among them J2 G125-MH104M4-04AD000P, U2 INA180, U3 SPX3819M5-L-1-2, U4 SPX3819M5-L-2-5, U5 LMR64010XMF, U6 SPX3819M5-L-3-3, U8 MCP1754S-3302xCB

Commit message: Fix Pranav review suggestions
Parts:
- R12: value 16.5mR -> 16mR
Changed lines of the file:
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@@
 			)
 		)
-		(property "Value" "16.5mR"
+		(property "Value" "16mR"
 			(at 73.66 28.8544 90)
 			(effects

Commit message: Fix review suggestions from non-fpga board
Parts:
- removed C21: 1uF, Capacitor_SMD:C_0805_2012Metric_Pad1.18x1.45mm_HandSolder, symbol Device:C
- removed L1: 12uH, Inductor_SMD:L_0805_2012Metric_Pad1.05x1.20mm_HandSolder, symbol Device:L
- removed TP2: 3V3D, TestPoint:TestPoint_Pad_1.5x1.5mm, symbol Connector:TestPoint
- removed U6: SPX3819M5-L-3-3, Package_TO_SOT_SMD:SOT-23-5_HandSoldering, symbol Regulator_Linear:SPX3819M5-L-3-3
- removed U8: MCP1754S-3302xCB, Package_TO_SOT_SMD:SOT-23, symbol Regulator_Linear:MCP1754S-3302xCB
- added L1: CC453232-120KL, ind:IND_BOURNS_CC453232, symbol ind:CC453232-120KL
- added L2: 1uH, symbol Device:L
- added R23: 453kR, symbol Device:R_US
- added R24: 100kR, symbol Device:R_US
- added U6: TLV62568ADRL, Package_TO_SOT_SMD:SOT-563, symbol Regulator_Switching:TLV62568ADRL
- added U8: SPX3819M5-L-3-3, Package_TO_SOT_SMD:SOT-23-5_HandSoldering, symbol Regulator_Linear:SPX3819M5-L-3-3
- C10: value 0.1uF -> 1uF
- C11: value 10nF -> 22uF; DigiKey 732-12169-1-ND -> (none)
- C13, C7: footprint Capacitor_SMD:C_0805_2012Metric_Pad1.18x1.45mm_HandSolder -> Capacitor_SMD:C_1210_3225Metric_Pad1.33x2.70mm_HandSolder
- C20: value 0.1uF -> 10nF
- C22: value 10uF -> 1uF
- C9: value 1uF -> 4.7uF; DigiKey 1276-6470-1-ND -> (none)
- F1: value 2A Polyfuse -> 0ZCG0075FF2C; footprint Fuse:Fuse_1206_3216Metric_Pad1.42x1.75mm_HandSolder -> Fuse:Fuse_1812_4532Metric_Pad1.30x3.40mm_HandSolder
- R12: value 16mR -> 25mR
Connections:
- net +3.3VA: now also U8.5 (OUT); no longer C20.1
- net +3V3: now also C11.1, L2.2, R23.1
- net +5V: now also L1.2, U6.3 (VIN), U6.5 (EN), U8.1 (IN), U8.3 (EN)
- net GND: now also R24.2, U6.2 (GND)
- net GNDA: now also U8.2 (GND)
- net at D1.2 (A), U5.1 (SW): now also L1.1
- new net: C20.1, U8.4 (BP)
- new net: L2.1, U6.4 (SW)
- new net: R23.2, R24.1, U6.1 (FB)
Other:
- note added: "GAIN: 100 V/V"
- note added: "https://webench.ti.com/appinfo/webench/scripts/SDP.cgi?ID=ACBD7DAB326D4695"
- note added: "https://webench.ti.com/appinfo/webench/scripts/SDP.cgi?ID=C736EEFC9B6D8E5C"
- note removed: "GAIN: 100 V/V = 40 dB"
- note removed: "WEBENCH 4.8-5.5 in, 24V out @ 75mA"
- note removed: "check these two"
- moved on the sheet: C1, C5, C6, TP3

Commit message: Fix layout errors after reviewing
Parts:
- L2: footprint (none) -> Inductor_SMD:L_1206_3216Metric_Pad1.22x1.90mm_HandSolder
- R23, R24: footprint (none) -> Resistor_SMD:R_0805_2012Metric_Pad1.20x1.40mm_HandSolder
Changed lines of the file:
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@@
 			)
 		)
-		(property "Footprint" ""
+		(property "Footprint" "Inductor_SMD:L_1206_3216Metric_Pad1.22x1.90mm_HandSolder"
 			(at 198.12 29.21 0)
 			(effects
@@
 			)
 		)
-		(property "Footprint" ""
+		(property "Footprint" "Resistor_SMD:R_0805_2012Metric_Pad1.20x1.40mm_HandSolder"
 			(at 210.566 34.544 90)
 			(effects
@@
 			)
 		)
-		(property "Footprint" ""
+		(property "Footprint" "Resistor_SMD:R_0805_2012Metric_Pad1.20x1.40mm_HandSolder"
 			(at 210.566 44.704 90)
 			(effects

Commit message: Fix diode
Parts:
- added TP2: 3V3, TestPoint:TestPoint_Pad_1.5x1.5mm, symbol Connector:TestPoint
- D1: footprint Diode_SMD:D_0805_2012Metric_Pad1.15x1.40mm_HandSolder -> dio:DIO_RB051MM_ROM
Connections:
- net +3V3: now also TP2.1
Changed lines of the file:
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@@
 	)
 	(junction
+		(at 228.6 29.21)
+		(diameter 0)
+		(color 0 0 0 0)
+	)
+	(junction
 		(at 207.01 135.89)
 		(diameter 0)
@@
 	(wire
 		(pts
+			(xy 228.6 29.21) (xy 223.52 29.21)
+		)
+		(stroke
+			(width 0)
+			(type default)
+		)
+	)
+	(wire
+		(pts
 			(xy 87.63 29.21) (xy 87.63 31.75)
 		)
@@
 	(wire
 		(pts
-			(xy 234.95 29.21) (xy 223.52 29.21)
+			(xy 234.95 29.21) (xy 228.6 29.21)
 		)
 		(stroke
@@
 	(wire
 		(pts
+			(xy 228.6 26.67) (xy 228.6 29.21)
+		)
+		(stroke
+			(width 0)
+			(type default)
+		)
+	)
+	(wire
+		(pts
 			(xy 87.63 149.86) (xy 87.63 152.4)
 		)
@@
 	)
 	(symbol
+		(lib_id "Connector:TestPoint")
+		(at 228.6 26.67 0)
+		(unit 1)
+		(exclude_from_sim no)
+		(in_bom yes)
+		(on_board yes)
+		(dnp no)
+		(property "Reference" "TP2"
+			(at 223.52 23.622 0)
+			(effects
+				(font
+					(size 1.27 1.27)
+				)
+				(justify left)
+			)
+		)
+		(property "Value" "3V3"
+			(at 223.52 26.162 0)
+			(effects
+				(font
+					(size 1.27 1.27)
+				)
+				(justify left)
+			)
+		)
+		(property "Footprint" "TestPoint:TestPoint_Pad_1.5x1.5mm"
+			(at 233.68 26.67 0)
+			(effects
+				(font
+					(size 1.27 1.27)
+				)
+				(hide yes)
+			)
+		)
+		(property "Datasheet" "~"
+			(at 233.68 26.67 0)
+			(effects
+				(font
+					(size 1.27 1.27)
+				)
+				(hide yes)
+			)
+		)
+		(property "Description" "test point"
+			(at 228.6 26.67 0)
+			(effects
+				(font
+					(size 1.27 1.27)
+				)
+				(hide yes)
+			)
+		)
+		(pin "1"
+		)
+		(instances
+			(project "FPGA-Lockin"
+				(path "/0d4da0fe-f3e4-47fc-a7f7-d58161fd7b20/6a7b816a-f907-4b8a-819a-c702a9816aaa"
+					(reference "TP2")
+					(unit 1)
+				)
+			)
+		)
+	)
+	(symbol
 		(lib_id "Device:C")
 		(at 161.29 77.47 0)
@@
 			)
 		)
-		(property "Footprint" "Diode_SMD:D_0805_2012Metric_Pad1.15x1.40mm_HandSolder"
+		(property "Footprint" "dio:DIO_RB051MM_ROM"
 			(at 67.31 132.08 0)
 			(effects

Commit message: Fix everything based on component availabilty
Parts:
- removed C6: 1uF, Capacitor_SMD:C_0805_2012Metric_Pad1.18x1.45mm_HandSolder, symbol Device:C
- removed U3: SPX3819M5-L-1-2, Package_TO_SOT_SMD:SOT-23-5, symbol Regulator_Linear:SPX3819M5-L-1-2
- added L3: 1uH, Inductor_SMD:L_1206_3216Metric_Pad1.22x1.90mm_HandSolder, symbol Device:L
- added R26, R27: 100kR, Resistor_SMD:R_0805_2012Metric_Pad1.20x1.40mm_HandSolder, symbol Device:R_US
- added U3: TLV62568ADRL, Package_TO_SOT_SMD:SOT-563, symbol Regulator_Switching:TLV62568ADRL
- C4: value 1uF -> 4.7uF
- C5: value 10nF -> 22uF; DigiKey 732-12169-1-ND -> (none)
Connections:
- net +1V2: now also C5.1, L3.2, R26.1
- net +2V5: no longer C4.1
- net +5V: now also C4.1, U3.3 (VIN), U3.5 (EN)
- net GND: now also R27.2, U3.2 (GND)
- new net: R26.2, R27.1, U3.1 (FB)
- new net: L3.1, U3.4 (SW)
Other:
- moved on the sheet: TP5
